Commit message: init

File: urdf/chassis.urdf.xacro (robot description, xacro)
@@ -33,3 +33,24 @@
     <child link="ugv_devkit_v1_chassis_link" />
   </joint>
+  <!-- Base footprint link -->
+  <link name="base_footprint"></link>
+  <joint name="base_footprint_joint" type="fixed">
+    <origin xyz="0.0 0.0 0.0" rpy="0 0 0" />
+    <parent link="base_link" />
+    <child link="base_footprint" />
+  </joint>
+  <!-- Laser link -->
+  <link name="base_laser"></link>
+  <joint name="laser_joint" type="fixed">
+    <origin xyz="0.0 0.0 0.3" rpy="0 0 0" />
+    <parent link="base_link" />
+    <child link="base_laser" />
+  </joint>
+  <!-- Camera link -->
+  <link name="camera_link"></link>
+  <joint name="camera_joint" type="fixed">
+    <origin xyz="0.25 0.0 0.0" rpy="0 0 0" />
+    <parent link="base_link" />
+    <child link="camera_link" />
+  </joint>
 </robot>
